Commit message: add and fix some description config

File: ros2_ws/src/myarm_description/urdf/myarm_m750_poe_v3_2.urdf (robot description, URDF)
Before this commit: robot myarm_m750, 11 links, 10 joints
Joints:
- joint left_gripper_joint: limit lower=0.0 upper=0.0345 effort=20.0 velocity=0.05 -> lower=0.0 upper=0.04 effort=20.0 velocity=0.05
- joint right_gripper_joint: limit lower=0.0 upper=0.0345 effort=20.0 velocity=0.05 -> lower=0.0 upper=0.04 effort=20.0 velocity=0.05
