Commit message: add replay old runs

File: ros2_ws/src/myarm_description/urdf/myarm_m750_application.urdf.xacro (robot description, xacro)
@@ -12,4 +12,6 @@
   <xacro:arg name="wrist_camera_xyz" default="0 0 0"/>
   <xacro:arg name="wrist_camera_rpy" default="0 0 0"/>
+  <xacro:arg name="wrist_camera_optical_xyz" default="0 0 0"/>
+  <xacro:arg name="wrist_camera_optical_rpy" default="-1.570796326794897 0 -1.570796326794897"/>
   <!-- Plain URDF on purpose: pycore and Pinocchio continue to consume it. -->
   <xacro:include filename="myarm_m750_poe_v3_2.urdf"/>
@@ -21,5 +23,7 @@
       mount_rpy="$(arg wrist_camera_mount_rpy)"
       camera_xyz="$(arg wrist_camera_xyz)"
-      camera_rpy="$(arg wrist_camera_rpy)"/>
+      camera_rpy="$(arg wrist_camera_rpy)"
+      optical_xyz="$(arg wrist_camera_optical_xyz)"
+      optical_rpy="$(arg wrist_camera_optical_rpy)"/>
   </xacro:if>
 </robot>

File: ros2_ws/src/myarm_description/urdf/myarm_m750_neugrasp.urdf.xacro (robot description, xacro)
@@ -6,11 +6,13 @@
   for pycore, Pinocchio and planning.  This profile can add only the fixed
   camera subtree needed by NeuGrasp.
-  The four transform arguments describe:
+  The generic profile arguments describe:
     gripper_base_link -> wrist_camera_mount_link : mount_xyz / mount_rpy
     wrist_camera_mount_link -> wrist_camera_link : camera_xyz / camera_rpy
-  wrist_camera_link -> wrist_camera_optical_frame is defined by the camera
-  macro using the ROS optical-frame convention.  A launch layer must read and
-  validate a named calibration file before passing these values.  In
-  particular, do not enable the camera with these zero defaults on hardware.
+    wrist_camera_link -> wrist_camera_optical_frame : optical_xyz / optical_rpy
+  ``logitech_c925_wrist_v1`` instead selects a named model profile: its
+  bracket, body offset and body->optical transform are fixed in separate
+  Xacro files.  A launch layer accepts only a known profile from a named
+  calibration record.  In particular, do not enable the generic profile with
+  zero defaults on hardware.
   Application scene frames (workspace, volume, scan targets, selected grasp)
   must not be added here: they belong to their runtime owners, not robot TF.
@@ -18,18 +20,31 @@
 <robot xmlns:xacro="http://www.ros.org/wiki/xacro" name="myarm_m750">
   <xacro:arg name="use_wrist_camera" default="false"/>
-  <!-- Compatibility names shared with myarm_m750_application.urdf.xacro. -->
+  <xacro:arg name="wrist_camera_profile" default="generic"/>
+  <!-- Generic-profile compatibility names shared with application Xacro. -->
   <xacro:arg name="wrist_camera_mount_xyz" default="0 0 0"/>
   <xacro:arg name="wrist_camera_mount_rpy" default="0 0 0"/>
   <xacro:arg name="wrist_camera_xyz" default="0 0 0"/>
   <xacro:arg name="wrist_camera_rpy" default="0 0 0"/>
+  <xacro:arg name="wrist_camera_optical_xyz" default="0 0 0"/>
+  <xacro:arg name="wrist_camera_optical_rpy" default="-1.570796326794897 0 -1.570796326794897"/>
+  <xacro:property name="camera_profile" value="$(arg wrist_camera_profile)"/>
   <!-- Keep the canonical kinematic source as a plain URDF. -->
   <xacro:include filename="myarm_m750_poe_v3_2.urdf"/>
   <xacro:include filename="xacro/sensors/wrist_camera.xacro"/>
+  <xacro:include filename="xacro/sensors/mounts/logitech_c925_wrist_mount.xacro"/>
+  <xacro:include filename="xacro/sensors/profiles/logitech_c925_wrist_camera.xacro"/>
   <xacro:if value="$(arg use_wrist_camera)">
-    <xacro:myarm_neugrasp_wrist_camera
-      mount_xyz="$(arg wrist_camera_mount_xyz)"
-      mount_rpy="$(arg wrist_camera_mount_rpy)"
-      camera_xyz="$(arg wrist_camera_xyz)"
-      camera_rpy="$(arg wrist_camera_rpy)"/>
+    <xacro:if value="${camera_profile == 'generic'}">
+      <xacro:myarm_neugrasp_wrist_camera
+        mount_xyz="$(arg wrist_camera_mount_xyz)"
+        mount_rpy="$(arg wrist_camera_mount_rpy)"
+        camera_xyz="$(arg wrist_camera_xyz)"
+        camera_rpy="$(arg wrist_camera_rpy)"
+        optical_xyz="$(arg wrist_camera_optical_xyz)"
+        optical_rpy="$(arg wrist_camera_optical_rpy)"/>
+    </xacro:if>
+    <xacro:if value="${camera_profile == 'logitech_c925_wrist_v1'}">
+      <xacro:myarm_neugrasp_logitech_c925_wrist_camera/>
+    </xacro:if>
   </xacro:if>
 </robot>

File: ros2_ws/src/myarm_description/urdf/xacro/sensors/wrist_camera.xacro (robot description, xacro)
@@ -5,5 +5,5 @@
     The transform chain is deliberately split so that the physical mounting
     calibration remains explicit:
-      parent_link -> wrist_camera_mount_link -> wrist_camera_link
+      parent_link -> mount link -> wrist_camera_link
                   -> wrist_camera_optical_frame
     ``mount_*`` is the calibrated bracket/mount transform.  ``camera_*`` is
@@ -16,16 +16,16 @@
     physical camera dimensions are available.
   -->
-  <xacro:macro name="myarm_wrist_camera"
-               params="parent_link mount_xyz:='0 0 0' mount_rpy:='0 0 0'
-                       camera_xyz:='0 0 0' camera_rpy:='0 0 0'">
-    <link name="wrist_camera_mount_link"/>
-    <joint name="gripper_to_wrist_camera_mount_joint" type="fixed">
-      <parent link="${parent_link}"/>
-      <child link="wrist_camera_mount_link"/>
-      <origin xyz="${mount_xyz}" rpy="${mount_rpy}"/>
-    </joint>
+  <xacro:macro name="myarm_camera_body_and_optical"
+               params="parent_link camera_xyz:='0 0 0' camera_rpy:='0 0 0'
+                       optical_xyz:='0 0 0'
+                       optical_rpy:='-1.570796326794897 0 -1.570796326794897'">
+    <!--
+      This part is intentionally independent from the mount.  A model profile
+      can provide a named, fixed mount while reusing the semantic body and
+      optical frame names consumed by camera nodes and NeuGrasp.
+    -->
     <link name="wrist_camera_link"/>
     <joint name="wrist_camera_mount_joint" type="fixed">
-      <parent link="wrist_camera_mount_link"/>
+      <parent link="${parent_link}"/>
       <child link="wrist_camera_link"/>
       <origin xyz="${camera_xyz}" rpy="${camera_rpy}"/>
@@ -35,6 +35,24 @@
       <parent link="wrist_camera_link"/>
       <child link="wrist_camera_optical_frame"/>
-      <origin xyz="0 0 0" rpy="-1.570796326794897 0 -1.570796326794897"/>
+      <origin xyz="${optical_xyz}" rpy="${optical_rpy}"/>
     </joint>
+  </xacro:macro>
+  <xacro:macro name="myarm_wrist_camera"
+               params="parent_link mount_xyz:='0 0 0' mount_rpy:='0 0 0'
+                       camera_xyz:='0 0 0' camera_rpy:='0 0 0'
+                       optical_xyz:='0 0 0'
+                       optical_rpy:='-1.570796326794897 0 -1.570796326794897'">
+    <link name="wrist_camera_mount_link"/>
+    <joint name="gripper_to_wrist_camera_mount_joint" type="fixed">
+      <parent link="${parent_link}"/>
+      <child link="wrist_camera_mount_link"/>
+      <origin xyz="${mount_xyz}" rpy="${mount_rpy}"/>
+    </joint>
+    <xacro:myarm_camera_body_and_optical
+      parent_link="wrist_camera_mount_link"
+      camera_xyz="${camera_xyz}"
+      camera_rpy="${camera_rpy}"
+      optical_xyz="${optical_xyz}"
+      optical_rpy="${optical_rpy}"/>
   </xacro:macro>
   <!--
@@ -45,5 +63,7 @@
   <xacro:macro name="myarm_neugrasp_wrist_camera"
                params="mount_xyz:='0 0 0' mount_rpy:='0 0 0'
-                       camera_xyz:='0 0 0' camera_rpy:='0 0 0'">
+                       camera_xyz:='0 0 0' camera_rpy:='0 0 0'
+                       optical_xyz:='0 0 0'
+                       optical_rpy:='-1.570796326794897 0 -1.570796326794897'">
     <xacro:myarm_wrist_camera
       parent_link="gripper_base_link"
@@ -51,5 +71,7 @@
       mount_rpy="${mount_rpy}"
       camera_xyz="${camera_xyz}"
-      camera_rpy="${camera_rpy}"/>
+      camera_rpy="${camera_rpy}"
+      optical_xyz="${optical_xyz}"
+      optical_rpy="${optical_rpy}"/>
   </xacro:macro>
 </robot>

Commit message: add demo camera stack in pycore and ros

File: ros2_ws/src/myarm_description/urdf/myarm_m750_application.urdf.xacro (robot description, xacro)
@@ -8,4 +8,5 @@
 <robot xmlns:xacro="http://www.ros.org/wiki/xacro" name="myarm_m750">
   <xacro:arg name="use_wrist_camera" default="false"/>
+  <xacro:arg name="wrist_camera_profile" default="generic"/>
   <xacro:arg name="wrist_camera_mount_xyz" default="0 0 0"/>
   <xacro:arg name="wrist_camera_mount_rpy" default="0 0 0"/>
@@ -14,16 +15,24 @@
   <xacro:arg name="wrist_camera_optical_xyz" default="0 0 0"/>
   <xacro:arg name="wrist_camera_optical_rpy" default="-1.570796326794897 0 -1.570796326794897"/>
+  <xacro:property name="camera_profile" value="$(arg wrist_camera_profile)"/>
   <!-- Plain URDF on purpose: pycore and Pinocchio continue to consume it. -->
   <xacro:include filename="myarm_m750_poe_v3_2.urdf"/>
   <xacro:include filename="xacro/sensors/wrist_camera.xacro"/>
+  <xacro:include filename="xacro/sensors/mounts/logitech_c925e_wrist_mount.xacro"/>
+  <xacro:include filename="xacro/sensors/profiles/logitech_c925e_wrist_camera.xacro"/>
   <xacro:if value="$(arg use_wrist_camera)">
-    <xacro:myarm_wrist_camera
-      parent_link="gripper_base_link"
-      mount_xyz="$(arg wrist_camera_mount_xyz)"
-      mount_rpy="$(arg wrist_camera_mount_rpy)"
-      camera_xyz="$(arg wrist_camera_xyz)"
-      camera_rpy="$(arg wrist_camera_rpy)"
-      optical_xyz="$(arg wrist_camera_optical_xyz)"
-      optical_rpy="$(arg wrist_camera_optical_rpy)"/>
+    <xacro:if value="${camera_profile == 'generic'}">
+      <xacro:myarm_wrist_camera
+        parent_link="gripper_base_link"
+        mount_xyz="$(arg wrist_camera_mount_xyz)"
+        mount_rpy="$(arg wrist_camera_mount_rpy)"
+        camera_xyz="$(arg wrist_camera_xyz)"
+        camera_rpy="$(arg wrist_camera_rpy)"
+        optical_xyz="$(arg wrist_camera_optical_xyz)"
+        optical_rpy="$(arg wrist_camera_optical_rpy)"/>
+    </xacro:if>
+    <xacro:if value="${camera_profile == 'logitech_c925e_wrist_v1'}">
+      <xacro:myarm_logitech_c925e_wrist_camera/>
+    </xacro:if>
   </xacro:if>
 </robot>

File: ros2_ws/src/myarm_description/urdf/myarm_m750_neugrasp.urdf.xacro (robot description, xacro)
@@ -10,5 +10,5 @@
     wrist_camera_mount_link -> wrist_camera_link : camera_xyz / camera_rpy
     wrist_camera_link -> wrist_camera_optical_frame : optical_xyz / optical_rpy
-  ``logitech_c925_wrist_v1`` instead selects a named model profile: its
+  ``logitech_c925e_wrist_v1`` instead selects a named model profile: its
   bracket, body offset and body->optical transform are fixed in separate
   Xacro files.  A launch layer accepts only a known profile from a named
@@ -32,6 +32,6 @@
   <xacro:include filename="myarm_m750_poe_v3_2.urdf"/>
   <xacro:include filename="xacro/sensors/wrist_camera.xacro"/>
-  <xacro:include filename="xacro/sensors/mounts/logitech_c925_wrist_mount.xacro"/>
-  <xacro:include filename="xacro/sensors/profiles/logitech_c925_wrist_camera.xacro"/>
+  <xacro:include filename="xacro/sensors/mounts/logitech_c925e_wrist_mount.xacro"/>
+  <xacro:include filename="xacro/sensors/profiles/logitech_c925e_wrist_camera.xacro"/>
   <xacro:if value="$(arg use_wrist_camera)">
     <xacro:if value="${camera_profile == 'generic'}">
@@ -44,6 +44,6 @@
         optical_rpy="$(arg wrist_camera_optical_rpy)"/>
     </xacro:if>
-    <xacro:if value="${camera_profile == 'logitech_c925_wrist_v1'}">
-      <xacro:myarm_neugrasp_logitech_c925_wrist_camera/>
+    <xacro:if value="${camera_profile == 'logitech_c925e_wrist_v1'}">
+      <xacro:myarm_logitech_c925e_wrist_camera/>
     </xacro:if>
   </xacro:if>
